Commit message: update aliengo urdfs

File: legged_gym/resources/robots/aliengo/urdf/aliengo.urdf (robot description, URDF)
Before this commit: robot aliengo, 31 links, 30 joints
Links:
- link FL_calf: geometry collision box size=0.25 0.0208 0.016; visual mesh filename=package://../meshes/calf.dae scale=1 1 1
- link FL_hip: geometry collision cylinder length=0.0418 radius=0.046; visual mesh filename=package://../meshes/hip.dae scale=1 1 1
- link FL_thigh: geometry collision box size=0.25 0.0374 0.043; visual mesh filename=package://../meshes/thigh.dae scale=1 1 1
- link FR_calf: geometry collision box size=0.25 0.0208 0.016; visual mesh filename=package://../meshes/calf.dae scale=1 1 1
- link FR_hip: geometry collision cylinder length=0.0418 radius=0.046; visual mesh filename=package://../meshes/hip.dae scale=1 1 1
- link FR_thigh: geometry collision box size=0.25 0.0374 0.043; visual mesh filename=package://../meshes/thigh_mirror.dae scale=1 1 1
- link RL_calf: geometry collision box size=0.25 0.0208 0.016; visual mesh filename=package://../meshes/calf.dae scale=1 1 1
- link RL_hip: geometry collision cylinder length=0.0418 radius=0.046; visual mesh filename=package://../meshes/hip.dae scale=1 1 1
- link RL_thigh: geometry collision box size=0.25 0.0374 0.043; visual mesh filename=package://../meshes/thigh.dae scale=1 1 1
- link RR_calf: geometry collision box size=0.25 0.0208 0.016; visual mesh filename=package://../meshes/calf.dae scale=1 1 1
- link RR_hip: geometry collision cylinder length=0.0418 radius=0.046; visual mesh filename=package://../meshes/hip.dae scale=1 1 1
- link RR_thigh: geometry collision box size=0.25 0.0374 0.043; visual mesh filename=package://../meshes/thigh_mirror.dae scale=1 1 1
- link imu_link: geometry collision box size=.001 .001 .001; visual box size=0.001 0.001 0.001
- link trunk: geometry collision box size=0.647 0.15 0.112; visual mesh filename=package://../meshes/trunk.dae scale=1 1 1
Joints:
- joint FL_calf_joint: limit lower=-2.775 upper=-0.611 effort=55 velocity=15.89 -> lower=-2.775073510670984 upper=-0.610865238 effort=55 velocity=15.89
- joint FL_hip_joint: limit lower=-0.873 upper=1.047 effort=44 velocity=20 -> lower=-0.872664626 upper=1.047197551 effort=44 velocity=20
- joint FL_thigh_joint: limit lower=-0.524 upper=3.927 effort=44 velocity=20 -> lower=-0.523598776 upper=3.926990817 effort=44 velocity=20
- joint FR_calf_joint: limit lower=-2.775 upper=-0.611 effort=55 velocity=15.89 -> lower=-2.775073510670984 upper=-0.610865238 effort=55 velocity=15.89
- joint FR_hip_joint: limit lower=-0.873 upper=1.047 effort=44 velocity=20 -> lower=-0.872664626 upper=1.047197551 effort=44 velocity=20
- joint FR_thigh_joint: limit lower=-0.524 upper=3.927 effort=44 velocity=20 -> lower=-0.523598776 upper=3.926990817 effort=44 velocity=20
- joint RL_calf_joint: limit lower=-2.775 upper=-0.611 effort=55 velocity=15.89 -> lower=-2.775073510670984 upper=-0.610865238 effort=55 velocity=15.89
- joint RL_hip_joint: limit lower=-0.873 upper=1.047 effort=44 velocity=20 -> lower=-0.872664626 upper=1.047197551 effort=44 velocity=20
- joint RL_thigh_joint: limit lower=-0.524 upper=3.927 effort=44 velocity=20 -> lower=-0.523598776 upper=3.926990817 effort=44 velocity=20
- joint RR_calf_joint: limit lower=-2.775 upper=-0.611 effort=55 velocity=15.89 -> lower=-2.775073510670984 upper=-0.610865238 effort=55 velocity=15.89
- joint RR_hip_joint: limit lower=-0.873 upper=1.047 effort=44 velocity=20 -> lower=-0.872664626 upper=1.047197551 effort=44 velocity=20
- joint RR_thigh_joint: limit lower=-0.524 upper=3.927 effort=44 velocity=20 -> lower=-0.523598776 upper=3.926990817 effort=44 velocity=20

File: legged_gym/resources/robots/aliengo/urdf/aliengo_bigAng.urdf (robot description, URDF)
Before this commit: robot aliengo, 31 links, 30 joints
Links:
- link FL_calf: geometry collision box size=0.25 0.0208 0.016; visual mesh filename=package://../meshes/calf.dae scale=1 1 1
- link FL_hip: geometry collision cylinder length=0.0418 radius=0.046; visual mesh filename=package://../meshes/hip.dae scale=1 1 1
- link FL_thigh: geometry collision box size=0.25 0.0374 0.043; visual mesh filename=package://../meshes/thigh.dae scale=1 1 1
- link FR_calf: geometry collision box size=0.25 0.0208 0.016; visual mesh filename=package://../meshes/calf.dae scale=1 1 1
- link FR_hip: geometry collision cylinder length=0.0418 radius=0.046; visual mesh filename=package://../meshes/hip.dae scale=1 1 1
- link FR_thigh: geometry collision box size=0.25 0.0374 0.043; visual mesh filename=package://../meshes/thigh_mirror.dae scale=1 1 1
- link RL_calf: geometry collision box size=0.25 0.0208 0.016; visual mesh filename=package://../meshes/calf.dae scale=1 1 1
- link RL_hip: geometry collision cylinder length=0.0418 radius=0.046; visual mesh filename=package://../meshes/hip.dae scale=1 1 1
- link RL_thigh: geometry collision box size=0.25 0.0374 0.043; visual mesh filename=package://../meshes/thigh.dae scale=1 1 1
- link RR_calf: geometry collision box size=0.25 0.0208 0.016; visual mesh filename=package://../meshes/calf.dae scale=1 1 1
- link RR_hip: geometry collision cylinder length=0.0418 radius=0.046; visual mesh filename=package://../meshes/hip.dae scale=1 1 1
- link RR_thigh: geometry collision box size=0.25 0.0374 0.043; visual mesh filename=package://../meshes/thigh_mirror.dae scale=1 1 1
- link trunk: geometry collision box size=0.647 0.15 0.112; visual mesh filename=package://../meshes/trunk.dae scale=1 1 1
Joints:
- joint FL_thigh_joint: limit lower=-3.141592654 upper=4.71238898 effort=35.278 velocity=20 -> lower=-2.094395102 upper=4.188790205 effort=35.278 velocity=20
- joint FR_thigh_joint: limit lower=-3.141592654 upper=4.71238898 effort=35.278 velocity=20 -> lower=-2.094395102 upper=4.188790205 effort=35.278 velocity=20
- joint RL_thigh_joint: limit lower=-3.141592654 upper=4.71238898 effort=35.278 velocity=20 -> lower=-2.094395102 upper=4.188790205 effort=35.278 velocity=20
- joint RR_thigh_joint: limit lower=-3.141592654 upper=4.71238898 effort=35.278 velocity=20 -> lower=-2.094395102 upper=4.188790205 effort=35.278 velocity=20

File: legged_gym/resources/robots/aliengo/urdf/aliengo_lidar.urdf (robot description, URDF)
Before this commit: robot aliengo, 32 links, 31 joints
Links:
- link FL_calf: geometry collision box size=0.25 0.0208 0.016; visual mesh filename=package://../meshes/calf.dae scale=0.028 0.028 0.028
- link FL_hip: geometry collision cylinder length=0.0418 radius=0.046; visual mesh filename=package://../meshes/hip.dae scale=1 1 1
- link FL_thigh: geometry collision box size=0.25 0.0374 0.043; visual mesh filename=package://../meshes/thigh.dae scale=1 1 1
- link FR_calf: geometry collision box size=0.25 0.0208 0.016; visual mesh filename=package://../meshes/calf.dae scale=0.028 0.028 0.028
- link FR_hip: geometry collision cylinder length=0.0418 radius=0.046; visual mesh filename=package://../meshes/hip.dae scale=1 1 1
- link FR_thigh: geometry collision box size=0.25 0.0374 0.043; visual mesh filename=package://../meshes/thigh_mirror.dae scale=1 1 1
- link RL_calf: geometry collision box size=0.25 0.0208 0.016; visual mesh filename=package://../meshes/calf.dae scale=0.028 0.028 0.028
- link RL_hip: geometry collision cylinder length=0.0418 radius=0.046; visual mesh filename=package://../meshes/hip.dae scale=1 1 1
- link RL_thigh: geometry collision box size=0.25 0.0374 0.043; visual mesh filename=package://../meshes/thigh.dae scale=1 1 1
- link RR_calf: geometry collision box size=0.25 0.0208 0.016; visual mesh filename=package://../meshes/calf.dae scale=0.028 0.028 0.028
- link RR_hip: geometry collision cylinder length=0.0418 radius=0.046; visual mesh filename=package://../meshes/hip.dae scale=1 1 1
- link RR_thigh: geometry collision box size=0.25 0.0374 0.043; visual mesh filename=package://../meshes/thigh_mirror.dae scale=1 1 1
- link trunk: geometry collision box size=0.647 0.15 0.112; visual mesh filename=package://../meshes/trunk.dae scale=1 1 1
Joints:
- joint FL_calf_joint: limit lower=-2.775 upper=-0.611 effort=55 velocity=15.89 -> lower=-2.775073510670984 upper=-0.610865238 effort=55 velocity=15.89
- joint FL_hip_joint: limit lower=-0.873 upper=1.047 effort=44 velocity=20 -> lower=-0.872664626 upper=1.047197551 effort=44 velocity=20
- joint FL_thigh_joint: limit lower=-0.524 upper=3.927 effort=44 velocity=20 -> lower=-0.523598776 upper=3.926990817 effort=44 velocity=20
- joint FR_calf_joint: limit lower=-2.775 upper=-0.611 effort=55 velocity=15.89 -> lower=-2.775073510670984 upper=-0.610865238 effort=55 velocity=15.89
- joint FR_hip_joint: limit lower=-0.873 upper=1.047 effort=44 velocity=20 -> lower=-0.872664626 upper=1.047197551 effort=44 velocity=20
- joint FR_thigh_joint: limit lower=-0.524 upper=3.927 effort=44 velocity=20 -> lower=-0.523598776 upper=3.926990817 effort=44 velocity=20
- joint RL_calf_joint: limit lower=-2.775 upper=-0.611 effort=55 velocity=15.89 -> lower=-2.775073510670984 upper=-0.610865238 effort=55 velocity=15.89
- joint RL_hip_joint: limit lower=-0.873 upper=1.047 effort=44 velocity=20 -> lower=-0.872664626 upper=1.047197551 effort=44 velocity=20
- joint RL_thigh_joint: limit lower=-0.524 upper=3.927 effort=44 velocity=20 -> lower=-0.523598776 upper=3.926990817 effort=44 velocity=20
- joint RR_calf_joint: limit lower=-2.775 upper=-0.611 effort=55 velocity=15.89 -> lower=-2.775073510670984 upper=-0.610865238 effort=55 velocity=15.89
- joint RR_hip_joint: limit lower=-0.873 upper=1.047 effort=44 velocity=20 -> lower=-0.872664626 upper=1.047197551 effort=44 velocity=20
- joint RR_thigh_joint: limit lower=-0.524 upper=3.927 effort=44 velocity=20 -> lower=-0.523598776 upper=3.926990817 effort=44 velocity=20
